File: hardware/pcb-main/kicad/led_controller.kicad_sch (KiCad schematic)
At the start: 5 parts, among them IC1 SN74AHCT125PWR

Commit message: Updated to use ultra simplified 3v buck converter
Parts:
- IC1: footprint SOP65P640X120-14N -> motion-play-footprints:SOP65P640X120-14N
Other:
- title: (none) -> Motion Play Main Board
Changed lines of the file:
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@@
 	(generator_version "9.0")
 	(paper "A4")
+	(title_block
+		(title "Motion Play Main Board")
+		(date "2025-09-07")
+		(rev "5.0")
+	)
 	(junction
 		(at 146.05 88.9)
@@
 			)
 		)
-		(property "Footprint" "SOP65P640X120-14N"
+		(property "Footprint" "motion-play-footprints:SOP65P640X120-14N"
 			(at 170.18 168.58 0)
 			(effects
