File: hardware/pcb-main/kicad/led_controller.kicad_sch (KiCad schematic)
At the start: 5 parts, among them IC1 SN74AHCT125PWR

Commit message: Generate ESP32-S3 schematic sheet and apply integration modifications
Phase 1c: created esp32_spec.json and generate_esp32_sheet.py to produce
esp32_s3.kicad_sch with WROOM-1 module, EN/boot circuits, USB series
resistors, decoupling caps, and status LED. All components annotated via
centralized annotate.py.

Phase 1d partial: esp32_integration.py placed AMS1117, USBLC6, power
switch, USB hierarchical labels on power_management sheet; added ESP32
sheet reference and removed U2/U1/unused test points from root sheet.

Fixed modify.py annotate.py path resolution bug. Fixed generator UUID
mismatch that caused kiutils to reset reference designators to '?'.

Made-with: Cursor
Changed lines of the file:
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@@
 					(size 1.27 1.27)
 				)
-				(hide yes)
 			)
 		)
@@
 					(size 1.27 1.27)
 				)
-				(hide yes)
 			)
 		)
@@
 					(size 1.27 1.27)
 				)
-				(hide yes)
 			)
 		)
@@
 					(size 1.27 1.27)
 				)
-				(hide yes)
 			)
 		)
@@
 					(size 1.27 1.27)
 				)
-				(hide yes)
 			)
 		)
@@
 					(size 1.27 1.27)
 				)
-				(hide yes)
 			)
 		)
@@
 					(size 1.27 1.27)
 				)
-				(hide yes)
 			)
 		)
@@
 					(size 1.27 1.27)
 				)
-				(hide yes)
 			)
 		)
@@
 					(size 1.27 1.27)
 				)
-				(hide yes)
 			)
 		)
@@
 					(size 1.27 1.27)
 				)
-				(hide yes)
 			)
 		)
@@
 					(size 1.27 1.27)
 				)
-				(hide yes)
 			)
 		)
@@
 					(size 1.27 1.27)
 				)
-				(hide yes)
 			)
 		)
@@
 					(size 1.27 1.27)
 				)
-				(hide yes)
 			)
 		)
@@
 					(size 1.27 1.27)
 				)
-				(hide yes)
 			)
 		)
@@
 					(size 1.27 1.27)
 				)
-				(hide yes)
 			)
 		)
@@
 					(size 1.27 1.27)
 				)
-				(hide yes)
 			)
 		)
@@
 					(size 1.27 1.27)
 				)
-				(hide yes)
 			)
 		)
@@
 					(size 1.27 1.27)
 				)
-				(hide yes)
 			)
 		)
@@
 					(size 1.27 1.27)
 				)
-				(hide yes)
 			)
 		)
@@
 					(size 1.27 1.27)
 				)
-				(hide yes)
 			)
 		)
@@
 					(size 1.27 1.27)
 				)
-				(hide yes)
 			)
 		)
@@
 					(size 1.27 1.27)
 				)
-				(hide yes)
 			)
 		)
@@
 					(size 1.27 1.27)
 				)
-				(hide yes)
 			)
 		)
@@
 					(size 1.27 1.27)
 				)
-				(hide yes)
 			)
 		)
@@
 					(size 1.27 1.27)
 				)
-				(hide yes)
 			)
 		)
@@
 					(size 1.27 1.27)
 				)
-				(hide yes)
 			)
 		)
@@
 					(size 1.27 1.27)
 				)
-				(hide yes)
 			)
 		)
@@
 					(size 1.27 1.27)
 				)
-				(hide yes)
 			)
 		)
@@
 					(size 1.27 1.27)
 				)
-				(hide yes)
 			)
 		)
@@
 					(size 1.27 1.27)
 				)
-				(hide yes)
 			)
 		)
@@
 					(size 1.27 1.27)
 				)
-				(hide yes)
 			)
 		)
@@
 					(size 1.27 1.27)
 				)
-				(hide yes)
 			)
 		)
@@
 					(size 1.27 1.27)
 				)
-				(hide yes)
 			)
 		)
@@
 				)
 				(justify left top)
-				(hide yes)
 			)
 		)
@@
 				)
 				(justify left top)
-				(hide yes)
 			)
 		)
@@
 					(size 1.27 1.27)
 				)
-				(hide yes)
 			)
 		)
@@
 				)
 				(justify left top)
-				(hide yes)
 			)
 		)
@@
 				)
 				(justify left top)
-				(hide yes)
 			)
 		)
@@
 				)
 				(justify left top)
-				(hide yes)
 			)
 		)
@@
 				)
 				(justify left top)
-				(hide yes)
 			)
 		)
@@
 				)
 				(justify left top)
-				(hide yes)
 			)
 		)
@@
 					(size 1.27 1.27)
 				)
-				(hide yes)
 			)
 		)
@@
 					(size 1.27 1.27)
 				)
-				(hide yes)
 			)
 		)
@@
 					(size 1.27 1.27)
 				)
-				(hide yes)
 			)
 		)
@@
 					(size 1.27 1.27)
 				)
-				(hide yes)
 			)
 		)
@@
 					(size 1.27 1.27)
 				)
-				(hide yes)
 			)
 		)
@@
 					(size 1.27 1.27)
 				)
-				(hide yes)
 			)
 		)
@@
 					(size 1.27 1.27)
 				)
-				(hide yes)
 			)
 		)
@@
 					(size 1.27 1.27)
 				)
-				(hide yes)
 			)
 		)
@@
 					(size 1.27 1.27)
 				)
-				(hide yes)
 			)
 		)
@@
 					(size 1.27 1.27)
 				)
-				(hide yes)
 			)
 		)
@@
 					(size 1.27 1.27)
 				)
-				(hide yes)
 			)
 		)
@@
 					(size 1.27 1.27)
 				)
-				(hide yes)
 			)
 		)
@@
 					(size 1.27 1.27)
 				)
-				(hide yes)
 			)
 		)
@@
 					(size 1.27 1.27)
 				)
-				(hide yes)
 			)
 		)
@@
 					(size 1.27 1.27)
 				)
-				(hide yes)
 			)
 		)
@@
 					(size 1.27 1.27)
 				)
-				(hide yes)
 			)
 		)
@@
 					(size 1.27 1.27)
 				)
-				(hide yes)
 			)
 		)
@@
 					(size 1.27 1.27)
 				)
-				(hide yes)
 			)
 		)
@@
 					(size 1.27 1.27)
 				)
-				(hide yes)
 			)
 		)
@@
 					(size 1.27 1.27)
 				)
-				(hide yes)
 			)
 		)
@@
 					(size 1.27 1.27)
 				)
-				(hide yes)
 			)
 		)
@@
 					(size 1.27 1.27)
 				)
-				(hide yes)
 			)
 		)
@@
 					(size 1.27 1.27)
 				)
-				(hide yes)
-			)
-		)
+			)
+		)

Commit message: Complete Phase 1d/1e: manual wiring, ERC clean (0 errors)
Root sheet:
- Wire ESP32_S3 sheet pins to system nets via labels (I2C_SDA,
  I2C_SCL, TCA_RESET, LED_DATA, CHRG_INT, USB_DP, USB_DN)
- Connect power pins with +3.3V, +5V, GND power symbols
- Add PWR_FLAG symbols to resolve power-not-driven ERC errors
- NC flags on INT1/2/3 (design decision to drop interrupt lines)
- Remove TPIO11/12/13 (INT test points, no longer needed)
- Clean up dangling wires from old U2/U1 area
- Remove stray I2C_SCL hierarchical label

Power management sheet:
- Wire J7 D+/D- pads (A6/B6 tied to USB_DP, A7/B7 tied to USB_DN)
- Insert VSYS_SW into power path: R44 and INA219 IN+ now on
  VSYS_SW net so SW1 actually disconnects boost converter input
- Position AMS1117, caps, USBLC6, power switch components

ESP32_S3 sheet:
- Add no-connect on D5 DOUT (status LED has no downstream chain)
- Component positioning cleanup

ERC: 0 errors, 69 warnings (all benign JLC-MCP pin type mismatches
and footprint library path issues)

Made-with: Cursor
Other:
- moved on the sheet: C7, C8, F1, IC1, R27
